File: demos/pic_programmer/pic_programmer.kicad_pcb (KiCad board)
At the start: 2 copper layers, 160 x 99.1 mm, 64 parts, among them J1 DB9-FEMAL, P1 CONN_2, P101 CONN_1, P102 CONN_1, P103 CONN_1, P104 CONN_1, P105 CONN_1, P106 CONN_1, P2 SUPP28, P3 SUPP40, Q1 BC237, Q2 BC307, Q3 BC307, U1 24Cxx, U2 74HC125, U3 7805, U4 LT1373, U5 PIC_18_PINS, U6 PIC_8_PINS

Commit message: demo update
Parts:
- removed REF**: TO-92, Package_TO_SOT_THT:TO-92
